File: r2/mega866.kicad_pcb (KiCad board)
At the start: 2 copper layers, 221.3 x 172.7 mm, 50 parts, among them J1 ZSM1-SM1, J10 Conn_01x06_Male, J11 Conn_01x02_Male, J12 Conn_01x02_Male, J2 ZSM1-SM2, J3 tl866_dip40, J4 Conn_01x06_Male, J5 tl866_dip40, J6 Conn_01x06_Male, J7 tl866_dip40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

Commit message: r2 sync
Signed-off-by: John McMaster <johndmcmaster@gmail.com>
Routing:
- net BPM_SR_CLK: track 89.9 -> 87.9 mm
- net BPM_SR_D: track 86.4 -> 84.7 mm
Other:
- board text added: "MEGA866 R2 (C) 2022 JOHN MCMASTER https://github.com/JohnDMcMaster/mega866-cad/"
- board text removed: "MEGA866 (C) 2022 JOHN MCMASTER https://github.com/JohnDMcMaster/mega866-cad/"
Changed lines of the file:
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@@
       (drillshape 0)
       (scaleselection 1)
-      (outputdirectory "mega866_r1")
+      (outputdirectory "mega866_r2")
     )
   )
@@
     (effects (font (size 2 2) (thickness 0.15)))
   )
-  (gr_text "MEGA866\n(C) 2022 JOHN MCMASTER\nhttps://github.com/JohnDMcMaster/mega866-cad/" (at 137.291309 167.64) (layer "F.SilkS")
+  (gr_text "MEGA866 R2\n(C) 2022 JOHN MCMASTER\nhttps://github.com/JohnDMcMaster/mega866-cad/" (at 137.291309 167.64) (layer "F.SilkS")
     (effects (font (size 2 2) (thickness 0.15)))
   )
@@
   (segment (start 100.25 119.925) (end 106.325 119.925) (width 0.19) (layer "B.Cu") (net 14))
   (segment (start 106.325 119.925) (end 124.575 101.675) (width 0.19) (layer "B.Cu") (net 14))
-  (segment (start 104 84.2245) (end 104 86) (width 0.19) (layer "F.Cu") (net 15))
+  (segment (start 102.729382 85.230618) (end 102.729382 119.090618) (width 0.19) (layer "F.Cu") (net 15))
   (segment (start 102.729382 119.090618) (end 99.06 122.76) (width 0.19) (layer "F.Cu") (net 15))
-  (segment (start 104 86) (end 102.729382 87.270618) (width 0.19) (layer "F.Cu") (net 15))
-  (segment (start 102.729382 87.270618) (end 102.729382 119.090618) (width 0.19) (layer "F.Cu") (net 15))
+  (segment (start 104 84.2245) (end 103.7355 84.2245) (width 0.19) (layer "F.Cu") (net 15))
+  (segment (start 103.7355 84.2245) (end 102.729382 85.230618) (width 0.19) (layer "F.Cu") (net 15))
   (via (at 104 84.2245) (size 0.8) (drill 0.4) (layers "F.Cu" "B.Cu") (net 15))
   (via (at 99.06 122.76) (size 0.8) (drill 0.4) (layers "F.Cu" "B.Cu") (net 15))
@@
   (segment (start 119.825 94.055) (end 114.775 94.055) (width 0.19) (layer "B.Cu") (net 37))
   (segment (start 121.475 94.055) (end 128.401309 94.055) (width 0.19) (layer "B.Cu") (net 38))
-  (segment (start 108 127.25) (end 108 70.75) (width 0.19) (layer "F.Cu") (net 42))
-  (segment (start 104.75 130.5) (end 108 127.25) (width 0.19) (layer "F.Cu") (net 42))
-  (segment (start 108 70.75) (end 109.5 69.25) (width 0.19) (layer "F.Cu") (net 42))
+  (segment (start 111.76 99.554867) (end 110.355 100.959867) (width 0.19) (layer "F.Cu") (net 42))
+  (segment (start 109.22 103.035133) (end 109.22 126.03) (width 0.19) (layer "F.Cu") (net 42))
+  (segment (start 110.355 100.959867) (end 110.355 101.900133) (width 0.19) (layer "F.Cu") (net 42))
+  (segment (start 111.76 69.85) (end 111.76 99.554867) (width 0.19) (layer "F.Cu") (net 42))
+  (segment (start 109.22 126.03) (end 104.75 130.5) (width 0.19) (layer "F.Cu") (net 42))
+  (segment (start 110.355 101.900133) (end 109.22 103.035133) (width 0.19) (layer "F.Cu") (net 42))
   (via (at 104.75 130.5) (size 0.8) (drill 0.4) (layers "F.Cu" "B.Cu") (net 42))
-  (via (at 109.5 69.25) (size 0.8) (drill 0.4) (layers "F.Cu" "B.Cu") (net 42))
+  (via (at 111.76 69.85) (size 0.8) (drill 0.4) (layers "F.Cu" "B.Cu") (net 42))
   (segment (start 101.075 130.5) (end 104.75 130.5) (width 0.19) (layer "B.Cu") (net 42))
   (segment (start 100.825 130.75) (end 101.075 130.5) (width 0.19) (layer "B.Cu") (net 42))
   (segment (start 127.806309 69.25) (end 128.401309 68.655) (width 0.19) (layer "B.Cu") (net 42))
-  (segment (start 109.5 69.25) (end 127.806309 69.25) (width 0.19) (layer "B.Cu") (net 42))
-  (segment (start 110.5 127.5) (end 108.25 129.75) (width 0.19) (layer "F.Cu") (net 43))
-  (segment (start 111 68.5) (end 110.5 69) (width 0.19) (layer "F.Cu") (net 43))
-  (segment (start 110.5 69) (end 110.5 127.5) (width 0.19) (layer "F.Cu") (net 43))
-  (via (at 111 68.5) (size 0.8) (drill 0.4) (layers "F.Cu" "B.Cu") (net 43))
+  (segment (start 111.76 69.85) (end 112.36 69.25) (width 0.19) (layer "B.Cu") (net 42))
+  (segment (start 112.36 69.25) (end 127.806309 69.25) (width 0.19) (layer "B.Cu") (net 42))
+  (segment (start 114.3 68.5655) (end 113.03 69.8355) (width 0.19) (layer "F.Cu") (net 43))
+  (segment (start 110.725 111.756263) (end 110.725 127.275) (width 0.19) (layer "F.Cu") (net 43))
+  (segment (start 113.03 109.451263) (end 110.725 111.756263) (width 0.19) (layer "F.Cu") (net 43))
+  (segment (start 113.03 69.8355) (end 113.03 109.451263) (width 0.19) (layer "F.Cu") (net 43))
+  (segment (start 110.725 127.275) (end 108.25 129.75) (width 0.19) (layer "F.Cu") (net 43))
+  (via (at 114.3 68.5655) (size 0.8) (drill 0.4) (layers "F.Cu" "B.Cu") (net 43))
   (via (at 108.25 129.75) (size 0.8) (drill 0.4) (layers "F.Cu" "B.Cu") (net 43))
-  (segment (start 113.385 66.115) (end 111 68.5) (width 0.19) (layer "B.Cu") (net 43))
-  (segment (start 128.401309 66.115) (end 113.385 66.115) (width 0.19) (layer "B.Cu") (net 43))
+  (segment (start 114.3 68.5655) (end 116.7505 66.115) (width 0.19) (layer "B.Cu") (net 43))
   (segment (start 104.25 133.75) (end 100.825 133.75) (width 0.19) (layer "B.Cu") (net 43))
   (segment (start 108.25 129.75) (end 104.25 133.75) (width 0.19) (layer "B.Cu") (net 43))
+  (segment (start 116.7505 66.115) (end 128.401309 66.115) (width 0.19) (layer "B.Cu") (net 43))
   (segment (start 113.9675 130.49) (end 113.9675 129.942683) (width 0.19) (layer "B.Cu") (net 64))
   (segment (start 113.9675 129.942683) (end 112.75 128.725183) (width 0.19) (layer "B.Cu") (net 64))
@@
   (segment (start 84.419 110.11) (end 87.92 110.11) (width 0.19) (layer "B.Cu") (net 132))
   (segment (start 78.263 116.266) (end 84.419 110.11) (width 0.19) (layer "B.Cu") (net 132))
-  (segment (start 64.643 159.766) (end 65.024 159.766) (width 0.19) (layer "B.Cu") (net 132))
   (segment (start 89.064 108.966) (end 90.043 108.966) (width 0.19) (layer "B.Cu") (net 132))
   (segment (start 65.024 159.766) (end 66.663 159.766) (width 0.19) (layer "B.Cu") (net 132))
